Commit message: Project Video changes

File: catkin_finalproj/src/drivers/universal_robot/ur_description/urdf/bottom_bun.urdf (robot description, URDF)
Before this commit: robot block, 1 links, 0 joints
Links:
- removed link burger_link
- added link bun_bottom_link, mass 0.02; collision mesh filename=package://ur_description/meshes/Bun_v3.stl scale=0.003 0.003 0.003; visual mesh filename=package://ur_description/meshes/Bun_v3.stl scale=0.003 0.003 0.003

File: catkin_finalproj/src/drivers/universal_robot/ur_description/urdf/cheese.urdf (robot description, URDF)
Before this commit: robot block, 1 links, 0 joints
Links:
- link cheese_link: geometry collision mesh filename=package://ur_description/meshes/cheese_v3.stl scale=0.003 0.003 0.005; visual mesh filename=package://ur_description/meshes/cheese_v3.stl scale=0.003 0.003 0.005

Commit message: Final full code push

File: catkin_finalproj/src/drivers/universal_robot/ur_description/urdf/bottom_bun.urdf (robot description, URDF)
Before this commit: robot block, 1 links, 0 joints
Links:
- link bun_bottom_link: geometry collision box size=0.075 0.075 0.020; visual mesh filename=package://ur_description/meshes/Bun_v3.stl scale=0.003 0.003 0.003

File: catkin_finalproj/src/drivers/universal_robot/ur_description/urdf/burger.urdf (robot description, URDF)
Before this commit: robot block, 1 links, 0 joints
Links:
- link burger_link: geometry collision box size=0.075 0.075 0.015; visual mesh filename=package://ur_description/meshes/burger_v1.stl scale=0.003 0.003 0.003

File: catkin_finalproj/src/drivers/universal_robot/ur_description/urdf/tomato.urdf (robot description, URDF)
Before this commit: robot block, 1 links, 0 joints
Links:
- removed link bun_link
- added link tom_link, mass 0.0225; collision box size=0.070 0.070 0.010; visual mesh filename=package://ur_description/meshes/burger_v1.stl scale=0.0025 0.0025 0.003
